Commit message: eqr_fix_urdf

File: resources/robots/eqr1_description/urdf/eqr1_pin.urdf (robot description, URDF)
Before this commit: robot eqr1, 17 links, 16 joints
Joints:
- removed joint fl_leg_1
- removed joint fl_leg_2
- removed joint fl_leg_3
- removed joint fr_leg_1
- removed joint fr_leg_2
- removed joint fr_leg_3
- removed joint hl_leg_1
- removed joint hl_leg_2
- removed joint hl_leg_3
- removed joint hr_leg_1
- removed joint hr_leg_2
- removed joint hr_leg_3
- added joint fl_leg_1_joint: type revolute, parent base_link, child fl_leg_l1, origin xyz=0.149 0.05 -0.045 rpy=0 0 0, axis 1 0 0, limit lower=-0.837 upper=0.837 effort=60 velocity=20
- added joint fl_leg_2_joint: type revolute, parent fl_leg_l1, child fl_leg_l2, origin xyz=0.0565 0 0 rpy=0 0 0, axis 0 1 0, limit lower=-3.49 upper=2.042 effort=60 velocity=20
- added joint fl_leg_3_joint: type revolute, parent fl_leg_l2, child fl_leg_l3, origin xyz=-0.19401 0.112 -0.048585 rpy=0 0 0, axis 0 1 0, limit lower=0 upper=1.84 effort=60 velocity=20
- added joint fr_leg_1_joint: type revolute, parent base_link, child fr_leg_l1, origin xyz=0.149 -0.05 -0.045 rpy=0 0 0, axis 1 0 0, limit lower=-0.837 upper=0.837 effort=60 velocity=20
- added joint fr_leg_2_joint: type revolute, parent fr_leg_l1, child fr_leg_l2, origin xyz=0.0565 0 0 rpy=0 0 0, axis 0 1 0, limit lower=-3.49 upper=2.042 effort=60 velocity=20
- added joint fr_leg_3_joint: type revolute, parent fr_leg_l2, child fr_leg_l3, origin xyz=-0.19401 -0.112 -0.048585 rpy=0 0 0, axis 0 1 0, limit lower=0 upper=1.84 effort=60 velocity=20
- added joint hl_leg_1_joint: type revolute, parent base_link, child hl_leg_l1, origin xyz=-0.149 0.05 -0.045 rpy=0 0 0, axis 1 0 0, limit lower=-0.837 upper=0.837 effort=60 velocity=20
- added joint hl_leg_2_joint: type revolute, parent hl_leg_l1, child hl_leg_l2, origin xyz=-0.0565 0 0 rpy=0 0 0, axis 0 1 0, limit lower=-3.49 upper=2.042 effort=60 velocity=20
- added joint hl_leg_3_joint: type revolute, parent hl_leg_l2, child hl_leg_l3, origin xyz=-0.19401 0.112 -0.048585 rpy=0 0 0, axis 0 1 0, limit lower=0 upper=1.84 effort=60 velocity=20
- added joint hr_leg_1_joint: type revolute, parent base_link, child hr_leg_l1, origin xyz=-0.149 -0.05 -0.045 rpy=0 0 0, axis 1 0 0, limit lower=-0.837 upper=0.837 effort=60 velocity=20
- added joint hr_leg_2_joint: type revolute, parent hr_leg_l1, child hr_leg_l2, origin xyz=-0.0565 0 0 rpy=0 0 0, axis 0 1 0, limit lower=-3.49 upper=2.042 effort=60 velocity=20
- added joint hr_leg_3_joint: type revolute, parent hr_leg_l2, child hr_leg_l3, origin xyz=-0.19401 -0.112 -0.048585 rpy=0 0 0, axis 0 1 0, limit lower=0 upper=1.84 effort=60 velocity=20

Commit message: fix urdf

File: resources/robots/eqr1_description/urdf/eqr1_pin.urdf (robot description, URDF)
Before this commit: robot eqr1, 17 links, 16 joints
Links:
- link fl_leg_l1: geometry collision mesh filename=../meshes/fl_leg_l1.STL; visual mesh filename=../meshes/fl_leg_l1.STL
- link fl_leg_l2: geometry collision mesh filename=../meshes/fl_leg_l2.STL; visual mesh filename=../meshes/fl_leg_l2.STL
- link fl_leg_l3: geometry collision mesh filename=../meshes/fl_leg_l3.STL; visual mesh filename=../meshes/fl_leg_l3.STL
- link fl_leg_lee: geometry collision mesh filename=../meshes/fl_leg_ee.STL; visual mesh filename=../meshes/fl_leg_ee.STL
- link fr_leg_l1: geometry collision mesh filename=../meshes/fr_leg_l1.STL; visual mesh filename=../meshes/fr_leg_l1.STL
- link fr_leg_l2: geometry collision mesh filename=../meshes/fr_leg_l2.STL; visual mesh filename=../meshes/fr_leg_l2.STL
- link fr_leg_l3: geometry collision mesh filename=../meshes/fr_leg_l3.STL; visual mesh filename=../meshes/fr_leg_l3.STL
- link hl_leg_l1: geometry collision mesh filename=../meshes/hl_leg_l1.STL; visual mesh filename=../meshes/hl_leg_l1.STL
- link hl_leg_l2: geometry collision mesh filename=../meshes/hl_leg_l2.STL; visual mesh filename=../meshes/hl_leg_l2.STL
- link hl_leg_l3: geometry collision mesh filename=../meshes/hl_leg_l3.STL; visual mesh filename=../meshes/hl_leg_l3.STL
- link hr_leg_l1: geometry collision mesh filename=../meshes/hr_leg_l1.STL; visual mesh filename=../meshes/hr_leg_l1.STL

Commit message: long way to go

File: resources/robots/eqr1_description/urdf/eqr1_pin.urdf (robot description, URDF)
Before this commit: robot eqr1, 17 links, 16 joints
Links:
- link fl_leg_l1: geometry collision cylinder length=0.146 radius=0.046; visual mesh filename=../meshes/fl_leg_l1.STL
- link fl_leg_l2: geometry collision box size=0.035 0.025 0.16; visual mesh filename=../meshes/fl_leg_l2.STL
- link fl_leg_l3: geometry collision box size=0.02 0.025 0.14; visual mesh filename=../meshes/fl_leg_l3.STL
- link fl_leg_lee: geometry collision sphere radius=0.022; visual mesh filename=../meshes/fl_leg_ee.STL
- link fr_leg_l1: geometry collision cylinder length=0.146 radius=0.046; visual mesh filename=../meshes/fr_leg_l1.STL
- link fr_leg_l2: geometry collision box size=0.035 0.025 0.16; visual mesh filename=../meshes/fr_leg_l2.STL
- link fr_leg_l3: geometry collision box size=0.02 0.025 0.14; visual mesh filename=../meshes/fr_leg_l3.STL
- link fr_leg_lee: geometry collision sphere radius=0.022; visual mesh filename=../meshes/fr_leg_ee.STL
- link hl_leg_l1: geometry collision cylinder length=0.146 radius=0.046; visual mesh filename=../meshes/hl_leg_l1.STL
- link hl_leg_l2: geometry collision box size=0.035 0.025 0.16; visual mesh filename=../meshes/hl_leg_l2.STL
- link hl_leg_l3: geometry collision box size=0.02 0.025 0.14; visual mesh filename=../meshes/hl_leg_l3.STL
- link hl_leg_lee: geometry collision sphere radius=0.022; visual mesh filename=../meshes/hl_leg_ee.STL
- link hr_leg_l1: geometry collision cylinder length=0.146 radius=0.046; visual mesh filename=../meshes/hr_leg_l1.STL
- link hr_leg_l2: geometry collision box size=0.035 0.025 0.16; visual mesh filename=../meshes/hr_leg_l2.STL
- link hr_leg_l3: geometry collision box size=0.02 0.025 0.14; visual mesh filename=../meshes/hr_leg_l3.STL
- link hr_leg_lee: geometry collision sphere radius=0.022; visual mesh filename=../meshes/hr_leg_ee.STL
